File: usb-type-c-breakout/usb-type-c-breakout.kicad_pcb (KiCad board)
At the start: 4 copper layers, 29.5 x 47.5 mm, 44 parts, among them J10 USB_B_Micro, J11 USB_C_Plug, J12 Conn_02x04_Odd_Even, J2 Conn_Coaxial, J3 Conn_Coaxial, J4 Conn_Coaxial, J5 Conn_Coaxial, J6 Conn_Coaxial, J7 Conn_Coaxial, J8 Conn_Coaxial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

Commit message: cleanup and BOM updates
Parts:
- added GS1: GS_logo-custom, Symbol:gs_logo_200mil, F.Cu at (100.0, 86.0)
Connections:
- net Net-(J10-Pad2) renamed /D-
- net Net-(J10-Pad3) renamed /D+
- net Net-(J11-PadA10) renamed /RX2-
- net Net-(J11-PadA11) renamed /RX2+
- net Net-(J11-PadA2) renamed /TX1+
- net Net-(J11-PadA3) renamed /TX1-
- net Net-(J11-PadA8) renamed /SBU1
- net Net-(J11-PadB10) renamed /RX1-
- net Net-(J11-PadB11) renamed /RX1+
- net Net-(J11-PadB2) renamed /TX2+
- net Net-(J11-PadB3) renamed /TX2-
- net Net-(J11-PadB5) renamed /VCONN
- net Net-(J11-PadB6) renamed /NC+
- net Net-(J11-PadB7) renamed /NC-
- net Net-(J11-PadB8) renamed /SBU2
Other:
- board text added: "Steiert Solutions"
- board text added: "USB Type-C Breakout"
