File: usb-type-c-breakout/usb-type-c-breakout.sch (KiCad schematic (older format))
At the start: 12 parts, among them J10 USB_B_Micro, J11 USB_C_Plug, J12 Conn_02x04_Odd_Even, J2 Conn_Coaxial, J3 Conn_Coaxial, J4 Conn_Coaxial, J5 Conn_Coaxial, J6 Conn_Coaxial, J7 Conn_Coaxial, J8 Conn_Coaxial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

Commit message: fully connected, with poured planes
Connections:
- net GND: now also J10.5 (GND), J10.6 (Shield), J2.2 (Ext), J3.2 (Ext), J4.2 (Ext), J5.2 (Ext), J6.2 (Ext), J7.2 (Ext), J8.2 (Ext), J9.2 (Ext)
Changed lines of the file:
@@
 Connection ~ 4600 4600
 Wire Wire Line
-	4600 4600 4400 4600
+	4600 4600 4500 4600
 Wire Wire Line
 	6200 2700 6500 2700
@@
 Connection ~ 6200 4850
 Wire Wire Line
-	6200 4850 2800 4850
+	6200 4850 4500 4850
 Wire Wire Line
 	6200 4750 6200 4850
@@
 Text Label 4650 1800 0    50   ~ 0
 CC
+Wire Wire Line
+	4500 4600 4500 4850
+Connection ~ 4500 4600
+Wire Wire Line
+	4500 4600 4400 4600
+Connection ~ 4500 4850
+Wire Wire Line
+	4500 4850 2800 4850
+Wire Wire Line
+	2500 3100 2500 4350
+Connection ~ 2500 3100
+Connection ~ 2500 4350
 $EndSCHEMATC

Commit message: cleanup and BOM updates
Parts:
- added GS1: GS_logo-custom, Symbol:gs_logo_200mil, symbol Graphic:GS_logo-custom
- J10: MFN (none) -> 629105150521; Mouser (none) -> 710-629105150521
- J11: symbol custom:USB_C_Plug -> usb-type-c-breakout-rescue:USB_C_Plug-custom; MFN (none) -> DX07VN24WA2C1568; Mouser (none) -> 656-DX07VN24WA2C1568
- J12: MFN (none) -> 10129383-908001ALF; Mouser (none) -> 649-1012938390801ALF
- J2, J3, J4, J5, J6, J7, J8, J9: MFN (none) -> CON-SMA-EDGE; Mouser (none) -> 223-CON-SMA-EDGE
- R1: MFN (none) -> CR0603-JW-563ELF; Mouser (none) -> 652-CR0603JW-563ELF
Connections:
- net TX1+: now reaches J11.A2 (TX1+), J2.1 (In)
- net TX1-: now reaches J11.A3 (TX1-), J3.1 (In)
- net RX2-: now reaches J11.A10 (RX2-), J4.1 (In)
- net RX2+: now reaches J11.A11 (RX2+), J5.1 (In)
- net TX2+: now reaches J11.B2 (TX2+), J6.1 (In)
- net TX2-: now reaches J11.B3 (TX2-), J7.1 (In)
- net RX1-: now reaches J11.B10 (RX1-), J8.1 (In)
- net RX1+: now reaches J11.B11 (RX1+), J9.1 (In)
- net D+: now reaches J10.3 (D+), J11.A6 (D+)
- net D-: now reaches J10.2 (D-), J11.A7 (D-)
- net SBU1: now reaches J11.A8 (SBU1), J12.8 (Pin_8)
- net VCONN: now reaches J11.B5 (VCONN), J12.3 (Pin_3)
- net NC+: now reaches J11.B6 (NC+), J12.1 (Pin_1)
- net NC-: now reaches J11.B7 (NC-), J12.2 (Pin_2)
- net SBU2: now reaches J11.B8 (SBU2), J12.4 (Pin_4)
Other:
- note added: "Steiert\nSolutions"
